File: hardware/pcb/vdar.kicad_pcb (KiCad board)
At the start: 2 copper layers, 94.5 x 97.8 mm, 26 parts, among them J1 USB C PD Board 12V 5A, J2 Optical Endstop, J3 Optical Endstop, J4 TF-LUNA, M1 Nema 17, M2 Nema 17, U1 ESP32-DEVKITC, U2 MP1584EN Buck Converter, U3 TMC2209_SILENTSTEPSTICK, U4 TMC2209_SILENTSTEPSTICK

Commit message: Add silkscreen to PCB
Other:
- board text added: "Credit: Ruby"
